File: cinnruler.kicad_pcb (KiCad board)
At the start: 2 copper layers, 85.6 x 54 mm, 22 parts

Commit message: Fix mils error
Signed-off-by: sanyue <sanyue7th@gmail.com>
Other:
- board text added: "x1in (1000mil)"
- board text removed: "x1in (100mil)"
