File: argb.kicad_sch (KiCad schematic)
At the start: 1 part

Commit message: layout
Signed-off-by: sanyue <sanyue7th@gmail.com>
Parts:
- removed D4: WS2813, LED_SMD:LED_WS2812_PLCC6_5.0x5.0mm_P1.6mm, symbol LED:WS2813
- added D10, D100, D101, D102, D103, D104, D105, D106, D107, D108, D109, D11, D110, D111, D112, D113, D114, D115, D116, D117, D118, D119, D12, D120, D121, D122, D123, D124, D125, D126, D127, D128, D129, D13, D130, D131, D132, D133, D134, D135, D136, D137, D138, D139, D14, D140, D141, D142, D143, D144, D145, D146, D147, D148, D149, D15, D150, D151, D152, D153, D154, D155, D156, D157, D158, D159, D16, D160, D161, D162, D163, D164, D165, D166, D167, D168, D169, D17, D170, D171, D172, D173, D174, D175, D176, D177, D178, D179, D18, D180, D181, D182, D183, D184, D185, D186, D187, D188, D189, D19, D190, D191, D192, D193, D194, D195, D196, D197, D198, D199, D20, D200, D201, D202, D203, D204, D205, D206, D207, D208, D209, D21, D210, D211, D212, D213, D214, D215, D216, D217, D218, D219, D22, D220, D221, D222, D223, D224, D225, D226, D227, D228, D229, D23, D230, D231, D232, D233, D234, D235, D236, D237, D238, D239, D24, D240, D241, D242, D243, D244, D245, D246, D247, D248, D249, D25, D250, D251, D252, D253, D254, D255, D256, D257, D258, D259, D26, D260, D261, D262, D263, D264, D265, D266, D267, D268, D269, D27, D270, D271, D272, D273, D274, D275, D276, D277, D278, D279, D28, D280, D281, D282, D283, D284, D285, D286, D287, D288, D289, D29, D290, D291, D292, D293, D294, D295, D296, D297, D298, D299, D3, D30, D300, D301, D302, D303, D304, D305, D306, D307, D308, D309, D31, D310, D311, D312, D313, D314, D315, D316, D317, D318, D319, D32, D320, D321, D322, D323, D324, D325, D326, D327, D328, D329, D33, D330, D331, D332, D333, D334, D335, D336, D337, D338, D339, D34, D340, D341, D342, D343, D344, D345, D346, D347, D348, D349, D35, D350, D351, D352, D353, D354, D355, D356, D357, D358, D359, D36, D360, D361, D362, D363, D364, D365, D366, D367, D368, D369, D37, D370, D371, D372, D373, D374, D375, D376, D377, D378, D379, D38, D380, D381, D382, D383, D384, D385, D386, D387, D388, D389, D39, D390, D391, D4, D40, D41, D42, D43, D44, D45, D46, D47, D48, D49, D5, D50, D51, D55, D56, D57, D58, D59, D6, D60, D61, D62, D63, D64, D65, D66, D67, D68, D69, D70, D71, D72, D73, D74, D75, D76, D77, D78, D79, D80, D81, D82, D83, D84, D85, D86, D87, D88, D89, D9, D90, D91, D92, D93, D94, D95, D96, D97, D98, D99: WS2812B-2020, LED_SMD:LED_WS2812B-2020_PLCC4_2.0x2.0mm, symbol LED:WS2812B-2020
Connections:
- net 5v: now also D10.4 (VDD), D100.4 (VDD), D101.4 (VDD), D102.4 (VDD), D103.4 (VDD), D104.4 (VDD), D105.4 (VDD), D106.4 (VDD), D107.4 (VDD), D108.4 (VDD), D109.4 (VDD), D11.4 (VDD), D110.4 (VDD), D111.4 (VDD), D112.4 (VDD), D113.4 (VDD), D114.4 (VDD), D115.4 (VDD), D116.4 (VDD), D117.4 (VDD), D118.4 (VDD), D119.4 (VDD), D12.4 (VDD), D120.4 (VDD), D121.4 (VDD), D122.4 (VDD), D123.4 (VDD), D124.4 (VDD), D125.4 (VDD), D126.4 (VDD), D127.4 (VDD), D128.4 (VDD), D129.4 (VDD), D13.4 (VDD), D130.4 (VDD), D131.4 (VDD), D132.4 (VDD), D133.4 (VDD), D134.4 (VDD), D135.4 (VDD), D136.4 (VDD), D137.4 (VDD), D138.4 (VDD), D139.4 (VDD), D14.4 (VDD), D140.4 (VDD), D141.4 (VDD), D142.4 (VDD), D143.4 (VDD), D144.4 (VDD), D145.4 (VDD), D146.4 (VDD), D147.4 (VDD), D148.4 (VDD), D149.4 (VDD), D15.4 (VDD), D150.4 (VDD), D151.4 (VDD), D152.4 (VDD), D153.4 (VDD), D154.4 (VDD), D155.4 (VDD), D156.4 (VDD), D157.4 (VDD), D158.4 (VDD), D159.4 (VDD), D16.4 (VDD), D160.4 (VDD), D161.4 (VDD), D162.4 (VDD), D163.4 (VDD), D164.4 (VDD), D165.4 (VDD), D166.4 (VDD), D167.4 (VDD), D168.4 (VDD), D169.4 (VDD), D17.4 (VDD), D170.4 (VDD), D171.4 (VDD), D172.4 (VDD), D173.4 (VDD), D174.4 (VDD), D175.4 (VDD), D176.4 (VDD), D177.4 (VDD), D178.4 (VDD), D179.4 (VDD), D18.4 (VDD), D180.4 (VDD), D181.4 (VDD), D182.4 (VDD), D183.4 (VDD), D184.4 (VDD), D185.4 (VDD), D186.4 (VDD), D187.4 (VDD), D188.4 (VDD), D189.4 (VDD), D19.4 (VDD), D190.4 (VDD), D191.4 (VDD), D192.4 (VDD), D193.4 (VDD), D194.4 (VDD), D195.4 (VDD), D196.4 (VDD), D197.4 (VDD), D198.4 (VDD), D199.4 (VDD), D20.4 (VDD), D200.4 (VDD), D201.4 (VDD), D202.4 (VDD), D203.4 (VDD), D204.4 (VDD), D205.4 (VDD), D206.4 (VDD), D207.4 (VDD), D208.4 (VDD), D209.4 (VDD), D21.4 (VDD), D210.4 (VDD), D211.4 (VDD), D212.4 (VDD), D213.4 (VDD), D214.4 (VDD), D215.4 (VDD), D216.4 (VDD), D217.4 (VDD), D218.4 (VDD), D219.4 (VDD), D22.4 (VDD), D220.4 (VDD), D221.4 (VDD), D222.4 (VDD), D223.4 (VDD), D224.4 (VDD), D225.4 (VDD), D226.4 (VDD), D227.4 (VDD), D228.4 (VDD), D229.4 (VDD), D23.4 (VDD), D230.4 (VDD), D231.4 (VDD), D232.4 (VDD), D233.4 (VDD), D234.4 (VDD), D235.4 (VDD), D236.4 (VDD), D237.4 (VDD), D238.4 (VDD), D239.4 (VDD), D24.4 (VDD), D240.4 (VDD), D241.4 (VDD), D242.4 (VDD), D243.4 (VDD), D244.4 (VDD), D245.4 (VDD), D246.4 (VDD), D247.4 (VDD), D248.4 (VDD), D249.4 (VDD), D25.4 (VDD), D250.4 (VDD), D251.4 (VDD), D252.4 (VDD), D253.4 (VDD), D254.4 (VDD), D255.4 (VDD), D256.4 (VDD), D257.4 (VDD), D258.4 (VDD), D259.4 (VDD), D26.4 (VDD), D260.4 (VDD), D261.4 (VDD), D262.4 (VDD), D263.4 (VDD), D264.4 (VDD), D265.4 (VDD), D266.4 (VDD), D267.4 (VDD), D268.4 (VDD), D269.4 (VDD), D27.4 (VDD), D270.4 (VDD), D271.4 (VDD), D272.4 (VDD), D273.4 (VDD), D274.4 (VDD), D275.4 (VDD), D276.4 (VDD), D277.4 (VDD), D278.4 (VDD), D279.4 (VDD), D28.4 (VDD), D280.4 (VDD), D281.4 (VDD), D282.4 (VDD), D283.4 (VDD), D284.4 (VDD), D285.4 (VDD), D286.4 (VDD), D287.4 (VDD), D288.4 (VDD), D289.4 (VDD), D29.4 (VDD), D290.4 (VDD), D291.4 (VDD), D292.4 (VDD), D293.4 (VDD), D294.4 (VDD), D295.4 (VDD), D296.4 (VDD), D297.4 (VDD), D298.4 (VDD), D299.4 (VDD), D3.4 (VDD), D30.4 (VDD), D300.4 (VDD), D301.4 (VDD), D302.4 (VDD), D303.4 (VDD), D304.4 (VDD), D305.4 (VDD), D306.4 (VDD), D307.4 (VDD), D308.4 (VDD), D309.4 (VDD), D31.4 (VDD), D310.4 (VDD), D311.4 (VDD), D312.4 (VDD), D313.4 (VDD), D314.4 (VDD), D315.4 (VDD), D316.4 (VDD), D317.4 (VDD), D318.4 (VDD), D319.4 (VDD), D32.4 (VDD), D320.4 (VDD), D321.4 (VDD), D322.4 (VDD), D323.4 (VDD), D324.4 (VDD), D325.4 (VDD), D326.4 (VDD), D327.4 (VDD), D328.4 (VDD), D329.4 (VDD), D33.4 (VDD), D330.4 (VDD), D331.4 (VDD), D332.4 (VDD), D333.4 (VDD), D334.4 (VDD), D335.4 (VDD), D336.4 (VDD), D337.4 (VDD), D338.4 (VDD), D339.4 (VDD), D34.4 (VDD), D340.4 (VDD), D341.4 (VDD), D342.4 (VDD), D343.4 (VDD), D344.4 (VDD), D345.4 (VDD), D346.4 (VDD), D347.4 (VDD), D348.4 (VDD), D349.4 (VDD), D35.4 (VDD), D350.4 (VDD), D351.4 (VDD), D352.4 (VDD), D353.4 (VDD), D354.4 (VDD), D355.4 (VDD), D356.4 (VDD), D357.4 (VDD), D358.4 (VDD), D359.4 (VDD), D36.4 (VDD), D360.4 (VDD), D361.4 (VDD), D362.4 (VDD), D363.4 (VDD), D364.4 (VDD), D365.4 (VDD), D366.4 (VDD), D367.4 (VDD), D368.4 (VDD), D369.4 (VDD), D37.4 (VDD), D370.4 (VDD), D371.4 (VDD), D372.4 (VDD), D373.4 (VDD), D374.4 (VDD), D375.4 (VDD), D376.4 (VDD), D377.4 (VDD), D378.4 (VDD), D379.4 (VDD), D38.4 (VDD), D380.4 (VDD), D381.4 (VDD), D382.4 (VDD), D383.4 (VDD), D384.4 (VDD), D385.4 (VDD), D386.4 (VDD), D387.4 (VDD), D388.4 (VDD), D389.4 (VDD), D39.4 (VDD), D390.4 (VDD), D391.4 (VDD), D4.4 (VDD), D40.4 (VDD), D41.4 (VDD), D42.4 (VDD), D43.4 (VDD), D44.4 (VDD), D45.4 (VDD), D46.4 (VDD), D47.4 (VDD), D48.4 (VDD), D49.4 (VDD), D5.4 (VDD), D50.4 (VDD), D51.4 (VDD), D55.4 (VDD), D56.4 (VDD), D57.4 (VDD), D58.4 (VDD), D59.4 (VDD), D6.4 (VDD), D60.4 (VDD), D61.4 (VDD), D62.4 (VDD), D63.4 (VDD), D64.4 (VDD), D65.4 (VDD), D66.4 (VDD), D67.4 (VDD), D68.4 (VDD), D69.4 (VDD), D70.4 (VDD), D71.4 (VDD), D72.4 (VDD), D73.4 (VDD), D74.4 (VDD), D75.4 (VDD), D76.4 (VDD), D77.4 (VDD), D78.4 (VDD), D79.4 (VDD), D80.4 (VDD), D81.4 (VDD), D82.4 (VDD), D83.4 (VDD), D84.4 (VDD), D85.4 (VDD), D86.4 (VDD), D87.4 (VDD), D88.4 (VDD), D89.4 (VDD), D9.4 (VDD), D90.4 (VDD), D91.4 (VDD), D92.4 (VDD), D93.4 (VDD), D94.4 (VDD), D95.4 (VDD), D96.4 (VDD), D97.4 (VDD), D98.4 (VDD), D99.4 (VDD)
- net din: now also D3.3 (DIN)
- new net: D305.1 (DOUT), D306.3 (DIN)
- new net: D304.1 (DOUT), D305.3 (DIN)
- new net: D390.1 (DOUT), D391.3 (DIN)
- new net: D72.1 (DOUT), D73.3 (DIN)
- new net: D71.1 (DOUT), D72.3 (DIN)
- new net: D175.1 (DOUT), D176.3 (DIN)
- new net: D174.1 (DOUT), D175.3 (DIN)
- new net: D355.1 (DOUT), D356.3 (DIN)
- new net: D354.1 (DOUT), D355.3 (DIN)
- new net: D92.1 (DOUT), D93.3 (DIN)
- new net: D91.1 (DOUT), D92.3 (DIN)
- new net: D231.1 (DOUT), D232.3 (DIN)
- new net: D230.1 (DOUT), D231.3 (DIN)
- new net: D62.1 (DOUT), D63.3 (DIN)
- new net: D61.1 (DOUT), D62.3 (DIN)
- new net: D323.1 (DOUT), D324.3 (DIN)
- new net: D322.1 (DOUT), D323.3 (DIN)
- new net: D238.1 (DOUT), D239.3 (DIN)
- new net: D237.1 (DOUT), D238.3 (DIN)
- new net: D209.1 (DOUT), D210.3 (DIN)
- new net: D208.1 (DOUT), D209.3 (DIN)
- new net: D239.1 (DOUT), D240.3 (DIN)
- new net: D387.1 (DOUT), D388.3 (DIN)
- new net: D386.1 (DOUT), D387.3 (DIN)
- new net: D146.1 (DOUT), D147.3 (DIN)
- new net: D145.1 (DOUT), D146.3 (DIN)
- new net: D119.1 (DOUT), D120.3 (DIN)
- new net: D118.1 (DOUT), D119.3 (DIN)
- new net: D144.1 (DOUT), D145.3 (DIN)
- new net: D350.1 (DOUT), D351.3 (DIN)
- new net: D349.1 (DOUT), D350.3 (DIN)
- new net: D104.1 (DOUT), D105.3 (DIN)
- new net: D103.1 (DOUT), D104.3 (DIN)
- new net: D166.1 (DOUT), D167.3 (DIN)
- new net: D165.1 (DOUT), D166.3 (DIN)
- new net: D148.1 (DOUT), D149.3 (DIN)
- new net: D147.1 (DOUT), D148.3 (DIN)
- new net: D358.1 (DOUT), D359.3 (DIN)
- new net: D357.1 (DOUT), D358.3 (DIN)
- new net: D114.1 (DOUT), D115.3 (DIN)
- new net: D113.1 (DOUT), D114.3 (DIN)
- new net: D190.1 (DOUT), D191.3 (DIN)
- new net: D189.1 (DOUT), D190.3 (DIN)
- new net: D127.1 (DOUT), D128.3 (DIN)
- new net: D126.1 (DOUT), D127.3 (DIN)
- new net: D233.1 (DOUT), D234.3 (DIN)
- new net: D232.1 (DOUT), D233.3 (DIN)
- new net: D200.1 (DOUT), D201.3 (DIN)
- new net: D199.1 (DOUT), D200.3 (DIN)
- new net: D370.1 (DOUT), D371.3 (DIN)
- new net: D369.1 (DOUT), D370.3 (DIN)
- new net: D63.1 (DOUT), D64.3 (DIN)
- new net: D246.1 (DOUT), D247.3 (DIN)
- new net: D245.1 (DOUT), D246.3 (DIN)
- new net: D205.1 (DOUT), D206.3 (DIN)
- new net: D204.1 (DOUT), D205.3 (DIN)
- new net: D51.1 (DOUT), D55.3 (DIN)
- new net: D50.1 (DOUT), D51.3 (DIN)
- new net: D303.1 (DOUT), D304.3 (DIN)
- new net: D302.1 (DOUT), D303.3 (DIN)
- new net: D352.1 (DOUT), D353.3 (DIN)
- new net: D351.1 (DOUT), D352.3 (DIN)
- new net: D19.1 (DOUT), D20.3 (DIN)
- new net: D18.1 (DOUT), D19.3 (DIN)
- new net: D319.1 (DOUT), D320.3 (DIN)
- new net: D318.1 (DOUT), D319.3 (DIN)
- new net: D326.1 (DOUT), D327.3 (DIN)
- new net: D325.1 (DOUT), D326.3 (DIN)
- new net: D374.1 (DOUT), D375.3 (DIN)
- new net: D373.1 (DOUT), D374.3 (DIN)
- new net: D185.1 (DOUT), D186.3 (DIN)
- new net: D184.1 (DOUT), D185.3 (DIN)
- new net: D212.1 (DOUT), D213.3 (DIN)
- new net: D211.1 (DOUT), D212.3 (DIN)
- new net: D198.1 (DOUT), D199.3 (DIN)
- new net: D197.1 (DOUT), D198.3 (DIN)
- new net: D310.1 (DOUT), D311.3 (DIN)
- new net: D309.1 (DOUT), D310.3 (DIN)
- new net: D33.1 (DOUT), D34.3 (DIN)
- new net: D32.1 (DOUT), D33.3 (DIN)
- new net: D366.1 (DOUT), D367.3 (DIN)
- new net: D365.1 (DOUT), D366.3 (DIN)
- new net: D346.1 (DOUT), D347.3 (DIN)
- new net: D345.1 (DOUT), D346.3 (DIN)
- new net: D48.1 (DOUT), D49.3 (DIN)
- new net: D47.1 (DOUT), D48.3 (DIN)
- new net: D70.1 (DOUT), D71.3 (DIN)
- new net: D69.1 (DOUT), D70.3 (DIN)
- new net: D46.1 (DOUT), D47.3 (DIN)
- new net: D16.1 (DOUT), D17.3 (DIN)
- new net: D15.1 (DOUT), D16.3 (DIN)
- new net: D41.1 (DOUT), D42.3 (DIN)
- new net: D40.1 (DOUT), D41.3 (DIN)
- new net: D17.1 (DOUT), D18.3 (DIN)
- new net: D280.1 (DOUT), D281.3 (DIN)
- new net: D279.1 (DOUT), D280.3 (DIN)
- new net: D124.1 (DOUT), D125.3 (DIN)
- new net: D123.1 (DOUT), D124.3 (DIN)
- new net: D347.1 (DOUT), D348.3 (DIN)
- new net: D289.1 (DOUT), D290.3 (DIN)
- new net: D288.1 (DOUT), D289.3 (DIN)
- new net: D385.1 (DOUT), D386.3 (DIN)
- new net: D109.1 (DOUT), D110.3 (DIN)
- new net: D108.1 (DOUT), D109.3 (DIN)
- new net: D260.1 (DOUT), D261.3 (DIN)
- new net: D259.1 (DOUT), D260.3 (DIN)
- new net: D192.1 (DOUT), D193.3 (DIN)
- new net: D191.1 (DOUT), D192.3 (DIN)
- new net: D243.1 (DOUT), D244.3 (DIN)
- new net: D242.1 (DOUT), D243.3 (DIN)
- new net: D78.1 (DOUT), D79.3 (DIN)
- new net: D77.1 (DOUT), D78.3 (DIN)
- new net: D353.1 (DOUT), D354.3 (DIN)
- new net: D306.1 (DOUT), D307.3 (DIN)
- new net: D360.1 (DOUT), D361.3 (DIN)
- new net: D359.1 (DOUT), D360.3 (DIN)
- new net: D376.1 (DOUT), D377.3 (DIN)
- new net: D375.1 (DOUT), D376.3 (DIN)
- new net: D169.1 (DOUT), D170.3 (DIN)
- new net: D168.1 (DOUT), D169.3 (DIN)
- new net: D292.1 (DOUT), D293.3 (DIN)
- new net: D291.1 (DOUT), D292.3 (DIN)
- new net: D227.1 (DOUT), D228.3 (DIN)
- new net: D226.1 (DOUT), D227.3 (DIN)
- new net: D12.1 (DOUT), D13.3 (DIN)
- new net: D11.1 (DOUT), D12.3 (DIN)
- new net: D27.1 (DOUT), D28.3 (DIN)
- new net: D26.1 (DOUT), D27.3 (DIN)
- new net: D167.1 (DOUT), D168.3 (DIN)
- new net: D89.1 (DOUT), D90.3 (DIN)
- new net: D88.1 (DOUT), D89.3 (DIN)
- new net: D372.1 (DOUT), D373.3 (DIN)
- new net: D371.1 (DOUT), D372.3 (DIN)
- new net: D106.1 (DOUT), D107.3 (DIN)
- new net: D105.1 (DOUT), D106.3 (DIN)
- new net: D80.1 (DOUT), D81.3 (DIN)
- new net: D79.1 (DOUT), D80.3 (DIN)
- new net: D301.1 (DOUT), D302.3 (DIN)
- new net: D321.1 (DOUT), D322.3 (DIN)
- new net: D320.1 (DOUT), D321.3 (DIN)
- new net: D324.1 (DOUT), D325.3 (DIN)
- new net: D96.1 (DOUT), D97.3 (DIN)
- new net: D95.1 (DOUT), D96.3 (DIN)
- new net: D128.1 (DOUT), D129.3 (DIN)
- new net: D64.1 (DOUT), D65.3 (DIN)
- new net: D60.1 (DOUT), D61.3 (DIN)
- new net: D59.1 (DOUT), D60.3 (DIN)
- new net: D368.1 (DOUT), D369.3 (DIN)
- new net: D344.1 (DOUT), D345.3 (DIN)
- new net: D343.1 (DOUT), D344.3 (DIN)
- new net: D140.1 (DOUT), D141.3 (DIN)
- new net: D139.1 (DOUT), D140.3 (DIN)
- new net: D327.1 (DOUT), D328.3 (DIN)
- new net: D216.1 (DOUT), D217.3 (DIN)
- new net: D215.1 (DOUT), D216.3 (DIN)
- new net: D313.1 (DOUT), D314.3 (DIN)
- new net: D312.1 (DOUT), D313.3 (DIN)
- new net: D45.1 (DOUT), D46.3 (DIN)
- new net: D222.1 (DOUT), D223.3 (DIN)
- new net: D221.1 (DOUT), D222.3 (DIN)
- new net: D122.1 (DOUT), D123.3 (DIN)
- new net: D131.1 (DOUT), D132.3 (DIN)
- new net: D130.1 (DOUT), D131.3 (DIN)
- new net: D284.1 (DOUT), D285.3 (DIN)
- new net: D283.1 (DOUT), D284.3 (DIN)
- new net: D171.1 (DOUT), D172.3 (DIN)
- new net: D170.1 (DOUT), D171.3 (DIN)
- new net: D264.1 (DOUT), D265.3 (DIN)
- new net: D263.1 (DOUT), D264.3 (DIN)
- new net: D129.1 (DOUT), D130.3 (DIN)
- new net: D21.1 (DOUT), D22.3 (DIN)
- new net: D20.1 (DOUT), D21.3 (DIN)
- new net: D228.1 (DOUT), D229.3 (DIN)
- new net: D31.1 (DOUT), D32.3 (DIN)
- new net: D287.1 (DOUT), D288.3 (DIN)
- new net: D87.1 (DOUT), D88.3 (DIN)
- new net: D85.1 (DOUT), D86.3 (DIN)
- new net: D84.1 (DOUT), D85.3 (DIN)
- new net: D100.1 (DOUT), D101.3 (DIN)
- new net: D100.3 (DIN), D99.1 (DOUT)
- new net: D4.1 (DOUT), D5.3 (DIN)
- new net: D3.1 (DOUT), D4.3 (DIN)
- new net: D5.1 (DOUT), D6.3 (DIN)
- new net: D187.1 (DOUT), D188.3 (DIN)
- new net: D186.1 (DOUT), D187.3 (DIN)
- new net: D364.1 (DOUT), D365.3 (DIN)
- new net: D295.1 (DOUT), D296.3 (DIN)
- new net: D294.1 (DOUT), D295.3 (DIN)
- new net: D348.1 (DOUT), D349.3 (DIN)
- new net: D155.1 (DOUT), D156.3 (DIN)
- new net: D154.1 (DOUT), D155.3 (DIN)
- new net: D67.1 (DOUT), D68.3 (DIN)
- new net: D66.1 (DOUT), D67.3 (DIN)
- new net: D93.1 (DOUT), D94.3 (DIN)
- new net: D98.1 (DOUT), D99.3 (DIN)
- new net: D207.1 (DOUT), D208.3 (DIN)
- new net: D229.1 (DOUT), D230.3 (DIN)
- new net: D253.1 (DOUT), D254.3 (DIN)
- new net: D252.1 (DOUT), D253.3 (DIN)
- new net: D225.1 (DOUT), D226.3 (DIN)
- new net: D224.1 (DOUT), D225.3 (DIN)
- new net: D90.1 (DOUT), D91.3 (DIN)
- new net: D213.1 (DOUT), D214.3 (DIN)
- new net: D110.1 (DOUT), D111.3 (DIN)
- new net: D136.1 (DOUT), D137.3 (DIN)
- new net: D135.1 (DOUT), D136.3 (DIN)
- new net: D195.1 (DOUT), D196.3 (DIN)
- new net: D194.1 (DOUT), D195.3 (DIN)
- new net: D356.1 (DOUT), D357.3 (DIN)
- new net: D157.1 (DOUT), D158.3 (DIN)
- new net: D156.1 (DOUT), D157.3 (DIN)
- new net: D183.1 (DOUT), D184.3 (DIN)
- new net: D182.1 (DOUT), D183.3 (DIN)
- new net: D206.1 (DOUT), D207.3 (DIN)
- new net: D210.1 (DOUT), D211.3 (DIN)
- new net: D34.1 (DOUT), D35.3 (DIN)
- new net: D334.1 (DOUT), D335.3 (DIN)
- new net: D333.1 (DOUT), D334.3 (DIN)
- new net: D249.1 (DOUT), D250.3 (DIN)
- new net: D248.1 (DOUT), D249.3 (DIN)
- new net: D367.1 (DOUT), D368.3 (DIN)
- new net: D150.1 (DOUT), D151.3 (DIN)
- new net: D149.1 (DOUT), D150.3 (DIN)
- new net: D290.1 (DOUT), D291.3 (DIN)
- new net: D193.1 (DOUT), D194.3 (DIN)
- new net: D137.1 (DOUT), D138.3 (DIN)
- new net: D202.1 (DOUT), D203.3 (DIN)
- new net: D201.1 (DOUT), D202.3 (DIN)
- new net: D112.1 (DOUT), D113.3 (DIN)
- new net: D111.1 (DOUT), D112.3 (DIN)
- new net: D315.1 (DOUT), D316.3 (DIN)
- new net: D314.1 (DOUT), D315.3 (DIN)
- new net: D141.1 (DOUT), D142.3 (DIN)
- new net: D162.1 (DOUT), D163.3 (DIN)
- new net: D161.1 (DOUT), D162.3 (DIN)
- new net: D180.1 (DOUT), D181.3 (DIN)
- new net: D179.1 (DOUT), D180.3 (DIN)
- new net: D49.1 (DOUT), D50.3 (DIN)
- new net: D94.1 (DOUT), D95.3 (DIN)
- new net: D81.1 (DOUT), D82.3 (DIN)
- new net: D262.1 (DOUT), D263.3 (DIN)
- new net: D261.1 (DOUT), D262.3 (DIN)
- new net: D296.1 (DOUT), D297.3 (DIN)
- new net: D86.1 (DOUT), D87.3 (DIN)
- new net: D223.1 (DOUT), D224.3 (DIN)
- new net: D176.1 (DOUT), D177.3 (DIN)
- new net: D117.1 (DOUT), D118.3 (DIN)
- new net: D181.1 (DOUT), D182.3 (DIN)
- new net: D13.1 (DOUT), D14.3 (DIN)
- new net: D36.1 (DOUT), D37.3 (DIN)
- new net: D35.1 (DOUT), D36.3 (DIN)
- new net: D138.1 (DOUT), D139.3 (DIN)
- new net: D329.1 (DOUT), D330.3 (DIN)
- new net: D328.1 (DOUT), D329.3 (DIN)
- new net: D65.1 (DOUT), D66.3 (DIN)
- new net: D153.1 (DOUT), D154.3 (DIN)
- new net: D177.1 (DOUT), D178.3 (DIN)
- new net: D125.1 (DOUT), D126.3 (DIN)
- new net: D29.1 (DOUT), D30.3 (DIN)
- new net: D28.1 (DOUT), D29.3 (DIN)
- new net: D173.1 (DOUT), D174.3 (DIN)
- new net: D172.1 (DOUT), D173.3 (DIN)
- new net: D214.1 (DOUT), D215.3 (DIN)
- new net: D163.1 (DOUT), D164.3 (DIN)
- new net: D39.1 (DOUT), D40.3 (DIN)
- new net: D38.1 (DOUT), D39.3 (DIN)
- new net: D382.1 (DOUT), D383.3 (DIN)
- new net: D381.1 (DOUT), D382.3 (DIN)
- new net: D44.1 (DOUT), D45.3 (DIN)
- new net: D43.1 (DOUT), D44.3 (DIN)
- new net: D299.1 (DOUT), D300.3 (DIN)
- new net: D298.1 (DOUT), D299.3 (DIN)
- new net: D361.1 (DOUT), D362.3 (DIN)
- new net: D282.1 (DOUT), D283.3 (DIN)
- new net: D281.1 (DOUT), D282.3 (DIN)
- new net: D68.1 (DOUT), D69.3 (DIN)
- new net: D56.1 (DOUT), D57.3 (DIN)
- new net: D55.1 (DOUT), D56.3 (DIN)
- new net: D240.1 (DOUT), D241.3 (DIN)
- new net: D102.1 (DOUT), D103.3 (DIN)
- new net: D297.1 (DOUT), D298.3 (DIN)
- new net: D244.1 (DOUT), D245.3 (DIN)
- new net: D143.1 (DOUT), D144.3 (DIN)
- new net: D14.1 (DOUT), D15.3 (DIN)
- new net: D160.1 (DOUT), D161.3 (DIN)
- new net: D159.1 (DOUT), D160.3 (DIN)
- new net: D42.1 (DOUT), D43.3 (DIN)
- new net: D276.1 (DOUT), D277.3 (DIN)
- new net: D275.1 (DOUT), D276.3 (DIN)
- new net: D293.1 (DOUT), D294.3 (DIN)
- new net: D236.1 (DOUT), D237.3 (DIN)
- new net: D115.1 (DOUT), D116.3 (DIN)
- new net: D389.1 (DOUT), D390.3 (DIN)
- new net: D388.1 (DOUT), D389.3 (DIN)
- new net: D384.1 (DOUT), D385.3 (DIN)
- new net: D23.1 (DOUT), D24.3 (DIN)
- new net: D22.1 (DOUT), D23.3 (DIN)
- new net: D83.1 (DOUT), D84.3 (DIN)
- new net: D82.1 (DOUT), D83.3 (DIN)
- new net: D134.1 (DOUT), D135.3 (DIN)
- new net: D133.1 (DOUT), D134.3 (DIN)
- new net: D270.1 (DOUT), D271.3 (DIN)
- new net: D269.1 (DOUT), D270.3 (DIN)
- new net: D332.1 (DOUT), D333.3 (DIN)
- new net: D188.1 (DOUT), D189.3 (DIN)
- new net: D57.1 (DOUT), D58.3 (DIN)
- new net: D380.1 (DOUT), D381.3 (DIN)
- new net: D278.1 (DOUT), D279.3 (DIN)
- new net: D277.1 (DOUT), D278.3 (DIN)
- new net: D337.1 (DOUT), D338.3 (DIN)
- new net: D336.1 (DOUT), D337.3 (DIN)
- new net: D76.1 (DOUT), D77.3 (DIN)
- new net: D75.1 (DOUT), D76.3 (DIN)
- new net: D331.1 (DOUT), D332.3 (DIN)
- new net: D330.1 (DOUT), D331.3 (DIN)
- new net: D73.1 (DOUT), D74.3 (DIN)
- new net: D235.1 (DOUT), D236.3 (DIN)
- new net: D251.1 (DOUT), D252.3 (DIN)
- new net: D250.1 (DOUT), D251.3 (DIN)
- new net: D274.1 (DOUT), D275.3 (DIN)
- new net: D273.1 (DOUT), D274.3 (DIN)
- new net: D286.1 (DOUT), D287.3 (DIN)
- new net: D285.1 (DOUT), D286.3 (DIN)
- new net: D10.1 (DOUT), D11.3 (DIN)
- new net: D379.1 (DOUT), D380.3 (DIN)
- new net: D378.1 (DOUT), D379.3 (DIN)
- new net: D116.1 (DOUT), D117.3 (DIN)
- new net: D311.1 (DOUT), D312.3 (DIN)
- new net: D151.1 (DOUT), D152.3 (DIN)
- new net: D308.1 (DOUT), D309.3 (DIN)
- new net: D335.1 (DOUT), D336.3 (DIN)
- new net: D74.1 (DOUT), D75.3 (DIN)
- new net: D97.1 (DOUT), D98.3 (DIN)
- new net: D120.1 (DOUT), D121.3 (DIN)
- new net: D340.1 (DOUT), D341.3 (DIN)
- new net: D339.1 (DOUT), D340.3 (DIN)
- new net: D258.1 (DOUT), D259.3 (DIN)
- new net: D58.1 (DOUT), D59.3 (DIN)
- new net: D271.1 (DOUT), D272.3 (DIN)
- new net: D152.1 (DOUT), D153.3 (DIN)
- new net: D101.1 (DOUT), D102.3 (DIN)
- new net: D257.1 (DOUT), D258.3 (DIN)
- new net: D256.1 (DOUT), D257.3 (DIN)
- new net: D383.1 (DOUT), D384.3 (DIN)
- new net: D241.1 (DOUT), D242.3 (DIN)
- new net: D24.1 (DOUT), D25.3 (DIN)
- new net: D255.1 (DOUT), D256.3 (DIN)
- new net: D254.1 (DOUT), D255.3 (DIN)
- new net: D37.1 (DOUT), D38.3 (DIN)
- new net: D247.1 (DOUT), D248.3 (DIN)
- new net: D265.1 (DOUT), D266.3 (DIN)
- new net: D178.1 (DOUT), D179.3 (DIN)
- new net: D158.1 (DOUT), D159.3 (DIN)
- new net: D300.1 (DOUT), D301.3 (DIN)
- new net: D10.3 (DIN), D9.1 (DOUT)
- new net: D363.1 (DOUT), D364.3 (DIN)
- new net: D362.1 (DOUT), D363.3 (DIN)
- new net: D30.1 (DOUT), D31.3 (DIN)
- new net: D377.1 (DOUT), D378.3 (DIN)
- new net: D266.1 (DOUT), D267.3 (DIN)
- new net: D203.1 (DOUT), D204.3 (DIN)
- new net: D307.1 (DOUT), D308.3 (DIN)
- new net: D196.1 (DOUT), D197.3 (DIN)
- new net: D317.1 (DOUT), D318.3 (DIN)
- new net: D272.1 (DOUT), D273.3 (DIN)
- new net: D268.1 (DOUT), D269.3 (DIN)
- new net: D267.1 (DOUT), D268.3 (DIN)
- new net: D338.1 (DOUT), D339.3 (DIN)
- new net: D218.1 (DOUT), D219.3 (DIN)
- new net: D217.1 (DOUT), D218.3 (DIN)
- new net: D220.1 (DOUT), D221.3 (DIN)
- new net: D219.1 (DOUT), D220.3 (DIN)
- new net: D107.1 (DOUT), D108.3 (DIN)
- new net: D316.1 (DOUT), D317.3 (DIN)
- new net: D341.1 (DOUT), D342.3 (DIN)
- new net: D142.1 (DOUT), D143.3 (DIN)
- new net: D164.1 (DOUT), D165.3 (DIN)
- new net: D234.1 (DOUT), D235.3 (DIN)
- new net: D132.1 (DOUT), D133.3 (DIN)
- new net: D342.1 (DOUT), D343.3 (DIN)
- new net: D121.1 (DOUT), D122.3 (DIN)
- new net: D25.1 (DOUT), D26.3 (DIN)
- new net: D6.1 (DOUT), D9.3 (DIN)
- new net GND: D10.2 (VSS), D100.2 (VSS), D101.2 (VSS), D102.2 (VSS), D103.2 (VSS), D104.2 (VSS), D105.2 (VSS), D106.2 (VSS), D107.2 (VSS), D108.2 (VSS), D109.2 (VSS), D11.2 (VSS), D110.2 (VSS), D111.2 (VSS), D112.2 (VSS), D113.2 (VSS), D114.2 (VSS), D115.2 (VSS), D116.2 (VSS), D117.2 (VSS), D118.2 (VSS), D119.2 (VSS), D12.2 (VSS), D120.2 (VSS), D121.2 (VSS), D122.2 (VSS), D123.2 (VSS), D124.2 (VSS), D125.2 (VSS), D126.2 (VSS), D127.2 (VSS), D128.2 (VSS), D129.2 (VSS), D13.2 (VSS), D130.2 (VSS), D131.2 (VSS), D132.2 (VSS), D133.2 (VSS), D134.2 (VSS), D135.2 (VSS), D136.2 (VSS), D137.2 (VSS), D138.2 (VSS), D139.2 (VSS), D14.2 (VSS), D140.2 (VSS), D141.2 (VSS), D142.2 (VSS), D143.2 (VSS), D144.2 (VSS), D145.2 (VSS), D146.2 (VSS), D147.2 (VSS), D148.2 (VSS), D149.2 (VSS), D15.2 (VSS), D150.2 (VSS), D151.2 (VSS), D152.2 (VSS), D153.2 (VSS), D154.2 (VSS), D155.2 (VSS), D156.2 (VSS), D157.2 (VSS), D158.2 (VSS), D159.2 (VSS), D16.2 (VSS), D160.2 (VSS), D161.2 (VSS), D162.2 (VSS), D163.2 (VSS), D164.2 (VSS), D165.2 (VSS), D166.2 (VSS), D167.2 (VSS), D168.2 (VSS), D169.2 (VSS), D17.2 (VSS), D170.2 (VSS), D171.2 (VSS), D172.2 (VSS), D173.2 (VSS), D174.2 (VSS), D175.2 (VSS), D176.2 (VSS), D177.2 (VSS), D178.2 (VSS), D179.2 (VSS), D18.2 (VSS), D180.2 (VSS), D181.2 (VSS), D182.2 (VSS), D183.2 (VSS), D184.2 (VSS), D185.2 (VSS), D186.2 (VSS), D187.2 (VSS), D188.2 (VSS), D189.2 (VSS), D19.2 (VSS), D190.2 (VSS), D191.2 (VSS), D192.2 (VSS), D193.2 (VSS), D194.2 (VSS), D195.2 (VSS), D196.2 (VSS), D197.2 (VSS), D198.2 (VSS), D199.2 (VSS), D20.2 (VSS), D200.2 (VSS), D201.2 (VSS), D202.2 (VSS), D203.2 (VSS), D204.2 (VSS), D205.2 (VSS), D206.2 (VSS), D207.2 (VSS), D208.2 (VSS), D209.2 (VSS), D21.2 (VSS), D210.2 (VSS), D211.2 (VSS), D212.2 (VSS), D213.2 (VSS), D214.2 (VSS), D215.2 (VSS), D216.2 (VSS), D217.2 (VSS), D218.2 (VSS), D219.2 (VSS), D22.2 (VSS), D220.2 (VSS), D221.2 (VSS), D222.2 (VSS), D223.2 (VSS), D224.2 (VSS), D225.2 (VSS), D226.2 (VSS), D227.2 (VSS), D228.2 (VSS), D229.2 (VSS), D23.2 (VSS), D230.2 (VSS), D231.2 (VSS), D232.2 (VSS), D233.2 (VSS), D234.2 (VSS), D235.2 (VSS), D236.2 (VSS), D237.2 (VSS), D238.2 (VSS), D239.2 (VSS), D24.2 (VSS), D240.2 (VSS), D241.2 (VSS), D242.2 (VSS), D243.2 (VSS), D244.2 (VSS), D245.2 (VSS), D246.2 (VSS), D247.2 (VSS), D248.2 (VSS), D249.2 (VSS), D25.2 (VSS), D250.2 (VSS), D251.2 (VSS), D252.2 (VSS), D253.2 (VSS), D254.2 (VSS), D255.2 (VSS), D256.2 (VSS), D257.2 (VSS), D258.2 (VSS), D259.2 (VSS), D26.2 (VSS), D260.2 (VSS), D261.2 (VSS), D262.2 (VSS), D263.2 (VSS), D264.2 (VSS), D265.2 (VSS), D266.2 (VSS), D267.2 (VSS), D268.2 (VSS), D269.2 (VSS), D27.2 (VSS), D270.2 (VSS), D271.2 (VSS), D272.2 (VSS), D273.2 (VSS), D274.2 (VSS), D275.2 (VSS), D276.2 (VSS), D277.2 (VSS), D278.2 (VSS), D279.2 (VSS), D28.2 (VSS), D280.2 (VSS), D281.2 (VSS), D282.2 (VSS), D283.2 (VSS), D284.2 (VSS), D285.2 (VSS), D286.2 (VSS), D287.2 (VSS), D288.2 (VSS), D289.2 (VSS), D29.2 (VSS), D290.2 (VSS), D291.2 (VSS), D292.2 (VSS), D293.2 (VSS), D294.2 (VSS), D295.2 (VSS), D296.2 (VSS), D297.2 (VSS), D298.2 (VSS), D299.2 (VSS), D3.2 (VSS), D30.2 (VSS), D300.2 (VSS), D301.2 (VSS), D302.2 (VSS), D303.2 (VSS), D304.2 (VSS), D305.2 (VSS), D306.2 (VSS), D307.2 (VSS), D308.2 (VSS), D309.2 (VSS), D31.2 (VSS), D310.2 (VSS), D311.2 (VSS), D312.2 (VSS), D313.2 (VSS), D314.2 (VSS), D315.2 (VSS), D316.2 (VSS), D317.2 (VSS), D318.2 (VSS), D319.2 (VSS), D32.2 (VSS), D320.2 (VSS), D321.2 (VSS), D322.2 (VSS), D323.2 (VSS), D324.2 (VSS), D325.2 (VSS), D326.2 (VSS), D327.2 (VSS), D328.2 (VSS), D329.2 (VSS), D33.2 (VSS), D330.2 (VSS), D331.2 (VSS), D332.2 (VSS), D333.2 (VSS), D334.2 (VSS), D335.2 (VSS), D336.2 (VSS), D337.2 (VSS), D338.2 (VSS), D339.2 (VSS), D34.2 (VSS), D340.2 (VSS), D341.2 (VSS), D342.2 (VSS), D343.2 (VSS), D344.2 (VSS), D345.2 (VSS), D346.2 (VSS), D347.2 (VSS), D348.2 (VSS), D349.2 (VSS), D35.2 (VSS), D350.2 (VSS), D351.2 (VSS), D352.2 (VSS), D353.2 (VSS), D354.2 (VSS), D355.2 (VSS), D356.2 (VSS), D357.2 (VSS), D358.2 (VSS), D359.2 (VSS), D36.2 (VSS), D360.2 (VSS), D361.2 (VSS), D362.2 (VSS), D363.2 (VSS), D364.2 (VSS), D365.2 (VSS), D366.2 (VSS), D367.2 (VSS), D368.2 (VSS), D369.2 (VSS), D37.2 (VSS), D370.2 (VSS), D371.2 (VSS), D372.2 (VSS), D373.2 (VSS), D374.2 (VSS), D375.2 (VSS), D376.2 (VSS), D377.2 (VSS), D378.2 (VSS), D379.2 (VSS), D38.2 (VSS), D380.2 (VSS), D381.2 (VSS), D382.2 (VSS), D383.2 (VSS), D384.2 (VSS), D385.2 (VSS), D386.2 (VSS), D387.2 (VSS), D388.2 (VSS), D389.2 (VSS), D39.2 (VSS), D390.2 (VSS), D391.2 (VSS), D4.2 (VSS), D40.2 (VSS), D41.2 (VSS), D42.2 (VSS), D43.2 (VSS), D44.2 (VSS), D45.2 (VSS), D46.2 (VSS), D47.2 (VSS), D48.2 (VSS), D49.2 (VSS), D5.2 (VSS), D50.2 (VSS), D51.2 (VSS), D55.2 (VSS), D56.2 (VSS), D57.2 (VSS), D58.2 (VSS), D59.2 (VSS), D6.2 (VSS), D60.2 (VSS), D61.2 (VSS), D62.2 (VSS), D63.2 (VSS), D64.2 (VSS), D65.2 (VSS), D66.2 (VSS), D67.2 (VSS), D68.2 (VSS), D69.2 (VSS), D70.2 (VSS), D71.2 (VSS), D72.2 (VSS), D73.2 (VSS), D74.2 (VSS), D75.2 (VSS), D76.2 (VSS), D77.2 (VSS), D78.2 (VSS), D79.2 (VSS), D80.2 (VSS), D81.2 (VSS), D82.2 (VSS), D83.2 (VSS), D84.2 (VSS), D85.2 (VSS), D86.2 (VSS), D87.2 (VSS), D88.2 (VSS), D89.2 (VSS), D9.2 (VSS), D90.2 (VSS), D91.2 (VSS), D92.2 (VSS), D93.2 (VSS), D94.2 (VSS), D95.2 (VSS), D96.2 (VSS), D97.2 (VSS), D98.2 (VSS), D99.2 (VSS)
