File: cinna-chan-light.kicad_sch (KiCad schematic)
At the start: 1 part, among them U3 ESP32-S3-WROOM-1

Commit message: layout
Signed-off-by: sanyue <sanyue7th@gmail.com>
Connections:
- net 3v3: now also U3.2 (3V3)
- net USB Data -: now reaches U3.13 (USB_D-)
- net USB Data +: now reaches U3.14 (USB_D+)
Other:
- removed sheet light_white
- note removed: "haihai cinnachan! lets make a basic board with an ESP32 this is a SoM with RF frontend and antenna built-in"
- note removed: "this is a heirarchal sheet. click it to enter it, and notice to the wire is connected between the sheet and here. right click the sheet and click sync sheet pin to add the remaining 2/4 labels here!"
- note removed: "this is a local label. it can be referenced anywhere. it's not best practice to use these when not scrictly necessary (ie for one-off signals) because then the namespace can get messy"
- note removed: "this is a local label. it connects nodes in the same sheet. outside this sheet, 3v3 is not connected to 3v3 local label here"
- moved on the sheet: U3
